Commit message: Ball model added. Also camera and ball added to rotors_desecription as well.

File: models/rotors_description/urdf/component_snippets.xacro (robot description, xacro)
@@ -32,4 +32,25 @@
     </gazebo>
   </xacro:macro>
+  <!-- Macro to add a ball. -->
+  <xacro:macro name="ball_macro"
+    params="namespace parent_link *origin">
+    <link name ="${namespace}/ball_link">
+      <pose>0 0 0 0 0 0</pose>
+      <visual>
+        <geometry>
+          <sphere radius="0.05"/>
+        </geometry>
+        <material name="green"/>
+      </visual>
+    </link>
+    <joint name="${namespace}/ball_joint" type="fixed">
+      <xacro:insert_block name="origin" />
+      <parent link="${parent_link}" />
+      <child link="${namespace}/ball_link" />
+    </joint>
+    <gazebo reference="${namespace}/ball_link">
+      <material>Gazebo/Green</material>
+    </gazebo>
+  </xacro:macro>
   <!-- Macro to add a camera. -->
   <xacro:macro name="camera_macro"
@@ -50,5 +71,5 @@
             <xacro:insert_block name="cylinder" />
           </geometry>
-          <material name="red" />
+          <material name="grey" />
         </visual>
       </xacro:if>
@@ -65,4 +86,5 @@
     </joint>
     <gazebo reference="${namespace}/camera_${camera_suffix}_link">
+      <material>Gazebo/Grey</material>
       <sensor type="camera" name="${namespace}_camera_${camera_suffix}">
         <update_rate>${frame_rate}</update_rate>
@@ -91,5 +113,5 @@
           <alwaysOn>true</alwaysOn>
           <updateRate>${frame_rate}</updateRate>
-          <cameraName>camera_${camera_suffix}</cameraName>
+          <cameraName>camera${camera_suffix}</cameraName>
           <imageTopicName>image_raw</imageTopicName>
           <cameraInfoTopicName>camera_info</cameraInfoTopicName>

File: models/rotors_description/urdf/iris_base.xacro (robot description, xacro)
@@ -23,4 +23,6 @@
   <xacro:arg name='enable_mavlink_interface' default='true' />
   <xacro:arg name='enable_wind' default='false' />
+  <xacro:arg name='camera' default='false' />
+  <xacro:arg name='ball' default='false' />
   <!-- The following causes segfault with multiple vehicles if defaults to true!!! -->
   <xacro:arg name='enable_ground_truth' default='false' />
@@ -92,4 +94,34 @@
     <origin xyz="0 0 0" rpy="0 0 0" />
   </xacro:imu_plugin_macro>
+  <xacro:if value="$(arg camera)">
+    <!-- Mount a Camera. -->
+    <xacro:camera_macro
+    namespace="${namespace}"
+    parent_link="base_link"
+    camera_suffix=""
+    frame_rate="30.0"
+    horizontal_fov="1.3962634"
+    image_width="640"
+    image_height="480"
+    image_format="R8G8B8"
+    min_distance="0.02"
+    max_distance="300"
+    noise_mean="0.0"
+    noise_stddev="0.007"
+    enable_visual="1"
+    >
+    <box size="0.02 0.02 0.02"/>
+    <origin xyz="0.080 0 0.045" rpy="0 0 0"/>
+    </xacro:camera_macro>
+  </xacro:if>
+  <xacro:if value="$(arg ball)">
+    <!-- Mount a Ball. -->
+    <xacro:ball_macro
+    namespace="${namespace}"
+    parent_link="base_link"
+    >
+    <origin xyz="0 0 0.102" rpy="0 0 0"/>
+    </xacro:ball_macro>
+  </xacro:if>
   <xacro:if value="$(arg enable_ground_truth)">
     <!-- Mount an IMU providing ground truth. -->
